File: Lab 1/Updated_board_schematic.kicad_sch (KiCad schematic)
At the start: 38 parts, among them J1 Power, J2 HEADER, J3 HEADER, J9 Conn_01x08_MountingPin, SW1 RESET, SW2 SW_SPST, U2 LM7805_TO220, U3 RS232, U4 74LS373, U5 ATF16V8B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

Commit message: Last last designs for ;ab1 part3 board circuit
Parts:
- C2: value 1 uf -> 10 uf
- R1: value 1K -> 10k
Connections:
- net GND: now also U5.11 (I9/OE)
- net XTAL_1: now also U5.1 (I/CLK)
Changed lines of the file:
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@@
 	(wire
 		(pts
+			(xy 110.49 168.91) (xy 120.65 168.91)
+		)
+		(stroke
+			(width 0)
+			(type default)
+		)
+	)
+	(wire
+		(pts
 			(xy 240.03 48.26) (xy 240.03 49.53)
 		)
@@
 		)
 	)
+	(wire
+		(pts
+			(xy 138.43 191.77) (xy 143.51 191.77)
+		)
+		(stroke
+			(width 0)
+			(type default)
+		)
+	)
 	(polyline
 		(pts
@@
 		)
 	)
+	(global_label "XTAL_1"
+		(shape input)
+		(at 110.49 168.91 180)
+		(fields_autoplaced yes)
+		(effects
+			(font
+				(size 1.27 1.27)
+			)
+			(justify right)
+		)
+		(property "Intersheetrefs" "${INTERSHEET_REFS}"
+			(at 101.0339 168.91 0)
+			(effects
+				(font
+					(size 1.27 1.27)
+				)
+				(justify right)
+				(hide yes)
+			)
+		)
+	)
 	(global_label "GND"
 		(shape input)
@@
 		)
 	)
+	(global_label "GND"
+		(shape input)
+		(at 143.51 191.77 0)
+		(fields_autoplaced yes)
+		(effects
+			(font
+				(size 1.27 1.27)
+			)
+			(justify left)
+		)
+		(property "Intersheetrefs" "${INTERSHEET_REFS}"
+			(at 150.3657 191.77 0)
+			(effects
+				(font
+					(size 1.27 1.27)
+				)
+				(justify left)
+				(hide yes)
+			)
+		)
+	)
 	(global_label "P2.5{slash}A13"
 		(shape input)
@@
 			)
 		)
-		(property "Value" "1K"
+		(property "Value" "10k"
 			(at 257.81 57.1499 0)
 			(effects
@@
 			)
 		)
-		(property "Value" "1 uf"
+		(property "Value" "10 uf"
 			(at 259.08 36.8299 0)
 			(effects
